Commit message: built model, also with actuator

File: catkin_ws/src/turtlebot3/turtlebot3_description/urdf/turtlebot3_ball_waffle_pi.urdf.xacro (robot description, xacro)
@@ -32,27 +32,70 @@
   </link>
   <!-- MY STUFF -->
-  <link name="second_link">
+  <link name="arm_link">
     <inertial>
         <mass value="0.18" />
         <inertia ixx="0.0002835" ixy="0.0" ixz="0.0" iyy="0.0002835" iyz="0.0" izz="0.000324" />
     </inertial>
-    <origin rpy="0.0 0.0 0.0" xyz="0.0 0.0 0.0" />
-    <collision>
-      <geometry>
-        <box size="0.05 0.05 0.15" />
-      </geometry>
-    </collision>
-    <visual>
-      <geometry>
-        <box size="0.05 0.05 0.15" />
-      </geometry>
-    </visual>
-  </link>
-  <joint name="base_to_second_joint" type="continuous">
-    <parent link="base_link"/>
-    <child link="second_link"/>
+    <origin rpy="0.0 0.0 0.0" xyz="0.0 0.0 0.16" />
+    <collision>
+      <geometry>
+        <cylinder length=".3" radius=".01" />
+      </geometry>
+    </collision>
+    <visual>
+      <geometry>
+        <cylinder length=".3" radius=".01" />
+      </geometry>
+    </visual>
+  </link>
+  <joint name="base_to_arm_joint" type="revolute">
+    <parent link="base_link"/>
+    <child link="arm_link"/>
+    <limit effort="1000.0" lower="0.0" upper="0.548" velocity="0.5"/>
+    <axis xyz="0 1 0"/>
+    <origin xyz="0.0 0.0 0.15" rpy="0.0 0.0 0.0"/>
+  </joint>
+  <link name="catcher_link">
+    <inertial>
+        <mass value="0.05" />
+        <inertia ixx="0.0002835" ixy="0.0" ixz="0.0" iyy="0.0002835" iyz="0.0" izz="0.000324" />
+    </inertial>
+    <origin rpy="0 1.57 0" xyz="0.0 0.0 0.0" />
+    <collision>
+      <geometry>
+        <mesh filename="package://fetch/tube.stl" scale="0.1 0.1 0.1"/>
+        <!-- <cylinder length=".1" radius=".03" /> -->
+      </geometry>
+    </collision>
+    <visual>
+      <origin rpy="0 1.57 0" xyz="0.0 0.0 0.0" />
+      <geometry>
+        <mesh filename="package://fetch/tube.stl" scale="0.1 0.1 0.1"/>
+        <!-- <cylinder length=".1" radius=".03" /> -->
+      </geometry>
+    </visual>
+  </link>
+  <joint name="arm_to_catcher_joint" type="continuous">
+    <parent link="arm_link"/>
+    <child link="catcher_link"/>
     <axis xyz="1 0 0"/>
-    <origin xyz="0.0 0.0 0.2" rpy="0.0 0.0 0.0"/>
-  </joint>
+    <origin xyz="0.0 0.0 0.17" rpy="0.0 0.0 0.0"/>
+  </joint>
+  <!-- ROS Control plugin for Gazebo -->
+  <gazebo>
+    <plugin name="gazebo_ros_control" filename="libgazebo_ros_control.so">
+      <robotNamespace>/simple_model</robotNamespace>
+    </plugin>
+  </gazebo>
+  <!-- transmission -->
+  <transmission name="base_to_arm_trans">
+    <type>transmission_interface/SimpleTransmission</type>
+    <actuator name="motor1">
+      <mechanicalReduction>1</mechanicalReduction>
+    </actuator>
+    <joint name="base_to_arm_joint">
+      <hardwareInterface>EffortJointInterface</hardwareInterface>
+    </joint>
+  </transmission>
   <!-- END MY STUFF -->
   <joint name="wheel_left_joint" type="continuous">

Commit message: detect circles works

File: catkin_ws/src/turtlebot3/turtlebot3_description/urdf/turtlebot3_ball_waffle_pi.urdf.xacro (robot description, xacro)
@@ -229,5 +229,5 @@
   </link>
   <joint name="camera_joint" type="fixed">
-    <origin xyz="0.073 -0.011 0.084" rpy="0 0 0"/>
+    <origin xyz="0.073 -0.011 0.184" rpy="0 0 0"/> <!--0.084 -->
     <parent link="base_link"/>
     <child link="camera_link"/>

Commit message: config changes

File: catkin_ws/src/turtlebot3/turtlebot3_description/urdf/turtlebot3_ball_waffle_pi.urdf.xacro (robot description, xacro)
@@ -52,5 +52,5 @@
     <parent link="base_link"/>
     <child link="arm_link"/>
-    <limit effort="1000.0" lower="0.0" upper="0.548" velocity="0.5"/>
+    <limit effort="1000.0" lower="0.0" upper="1.57" velocity="0.5"/>
     <axis xyz="0 1 0"/>
     <origin xyz="0.0 0.0 0.15" rpy="0.0 0.0 0.0"/>
@@ -64,5 +64,5 @@
     <collision>
       <geometry>r
-        <mesh filename="package://fetch/tube.stl" scale="0.2 0.2 0.2"/>
+        <mesh filename="package://fetch/tube.stl" scale="0.4 0.4 0.4"/>
         <!-- <cylinder length=".1" radius=".03" /> -->
       </geometry>
@@ -71,5 +71,5 @@
       <origin rpy="0 1.57 0" xyz="0.0 0.0 0.0" />
       <geometry>
-        <mesh filename="package://fetch/tube.stl" scale="0.2 0.2 0.2"/>
+        <mesh filename="package://fetch/tube.stl" scale="0.4 0.4 0.4"/>
         <!-- <cylinder length=".1" radius=".03" /> -->
       </geometry>
@@ -80,5 +80,5 @@
     <child link="catcher_link"/>
     <axis xyz="1 0 0"/>
-    <origin xyz="-0.04 0.0 0.23" rpy="0.0 0.0 0.0"/>
+    <origin xyz="-0.04 0.0 0.28" rpy="0.0 0.0 0.0"/>
   </joint>
   <!-- ROS Control plugin for Gazebo -->

Commit message: first test case works

File: catkin_ws/src/turtlebot3/turtlebot3_description/urdf/turtlebot3_ball_waffle_pi.urdf.xacro (robot description, xacro)
@@ -52,24 +52,31 @@
     <parent link="base_link"/>
     <child link="arm_link"/>
-    <limit effort="1000.0" lower="0.0" upper="1.57" velocity="0.5"/>
+    <limit effort="1000.0" lower="-1.57" upper=".3" velocity="0.5"/>
     <axis xyz="0 1 0"/>
-    <origin xyz="0.0 0.0 0.15" rpy="0.0 0.0 0.0"/>
+    <origin xyz="-0.14 0.0 0.15" rpy="0.0 0.0 0.0"/>
   </joint>
   <link name="catcher_link">
     <inertial>
-        <mass value="0.05" />
+        <mass value="0.001" />
         <inertia ixx="0.0002835" ixy="0.0" ixz="0.0" iyy="0.0002835" iyz="0.0" izz="0.000324" />
     </inertial>
     <origin rpy="0 1.57 0" xyz="0.0 0.0 0.0" />
     <collision>
-      <geometry>r
-        <mesh filename="package://fetch/tube.stl" scale="0.4 0.4 0.4"/>
+      <origin rpy="0 1.57 0" xyz="0.0 0.0 0.0" />
+      <geometry>
+        <mesh filename="package://fetch/tube.stl" scale="0.4 0.4 0.3"/>
         <!-- <cylinder length=".1" radius=".03" /> -->
       </geometry>
+      <surface>
+        <friction>
+          <mu>0.01</mu>
+          <mu2>0.01</mu2>
+        </friction>
+      </surface>
     </collision>
     <visual>
       <origin rpy="0 1.57 0" xyz="0.0 0.0 0.0" />
       <geometry>
-        <mesh filename="package://fetch/tube.stl" scale="0.4 0.4 0.4"/>
+        <mesh filename="package://fetch/tube.stl" scale="0.4 0.4 0.3"/>
         <!-- <cylinder length=".1" radius=".03" /> -->
       </geometry>
@@ -80,5 +87,5 @@
     <child link="catcher_link"/>
     <axis xyz="1 0 0"/>
-    <origin xyz="-0.04 0.0 0.28" rpy="0.0 0.0 0.0"/>
+    <origin xyz="-.11 0.0 0.28" rpy="0.0 0.0 0.0"/>
   </joint>
   <!-- ROS Control plugin for Gazebo -->

File: catkin_ws/src/turtlebot3/turtlebot3_description/urdf/turtlebot3_waffle_pi.gazebo.xacro (robot description, xacro)
@@ -118,5 +118,5 @@
         </scan>
         <range>
-          <min>0.120</min>
+          <min>0.30</min> <!-- .12 -->
           <max>3.5</max>
           <resolution>0.015</resolution>
